File: kicad_files/hardware_challenge.kicad_pcb (KiCad board)
At the start: 4 copper layers, 61 x 71 mm, 25 parts, among them J1 12V INPUT, J3 Cable header, Q1 SiSS27DN, SW1 TEST BUTTON, U1 L7805, U2 Teensy4.1, U3 NEO-M8N, U4 CY8C9560A-24AXIT, U5 MAX2679

Commit message: Preliminary run thought. Nice and quick. Hitting mostly the hardware, with a hint of the software.
Parts:
- moved C6 0.72 mm to (148.2, 66.5)
Connections:
- R3 pad 1: GND -> +3.3V
- U3 pad 7: GND -> +3.3V
Routing:
- net +3.3V: track 10.6 -> 12.9 mm, vias 5 -> 6
- net +12V: track 6.20 -> 7.10 mm
- net CBL_2: track 16.2 -> 15.4 mm
- net Net-(U3-VCC_RF): track 17.8 -> 17.1 mm
- net UBX-TIMEPULSE: track 45.1 -> 44.5 mm
