File: kicad_files/hardware_challenge.kicad_sch (KiCad schematic)
At the start: 25 parts, among them J1 12V INPUT, J3 Cable header, Q1 SiSS27DN, SW1 TEST BUTTON, U1 L7805, U2 Teensy4.1, U3 NEO-M8N, U4 CY8C9560A-24AXIT, U5 MAX2679

Commit message: Preliminary run thought. Nice and quick. Hitting mostly the hardware, with a hint of the software.
Parts:
- added R5: 25k, symbol Device:R_Small
Connections:
- net +3.3V: now also R3.1, U3.7 (VDD_USB)
- net GND: no longer R3.1, U3.7 (VDD_USB)
- net at U3.11 (RF_IN): now also U5.A2, R5.2; no longer C5.1
- net at U3.14 (LNA_EN): now also R5.1
- net at L1.2: now also AE1.1 (A); no longer U5.A2
- net at U5.B1: now also C5.1; no longer AE1.1 (A)
- no-connect marks 75 -> 78
Other:
- moved on the sheet: AE1, C6, U5
